File: atlas.kicad_sch (KiCad schematic)
At the start: 39 parts, among them U2 TMS570LC43, U50 CAN_TRANSIEVER_MODULE, U51 CAN_TRANSIEVER_MODULE

Commit message: kasalarin connectorleri eklendi genel duzenlemeler yapildi.
Parts:
- added CN? (x2): DIN-2, symbol atlas_robot:DIN-2
- added J? (x3): DIN-4, symbol Connector:DIN-4
- added J? (x3): RJ45, symbol Connector:RJ45
- added J? (x2): DIN-3, symbol Connector:DIN-3
- added J?: DIN-7_CenterPin7, symbol Connector:DIN-7_CenterPin7
- added J?: DB9_Female, Connector_Dsub:DSUB-9_Female_Horizontal_P2.77x2.84mm_EdgePinOffset9.40mm, symbol Connector:DB9_Female
- added J?: DIN-5, symbol Connector:DIN-5
- added J?: DIN-6, symbol Connector:DIN-6
- added U?: Ethernet_Switch, symbol atlas:Ethernet_Switch
- added U?: IO_Case, symbol atlas:IO_Case
- added U?: traktor_cn_5, symbol atlas:traktor_cn_5
- added U?: traktor_pow_cn, symbol atlas:traktor_pow_cn
Other:
- note added: "IO CONNECTION"
- note removed: "IOS CONNECTION"
- moved on the sheet: BTN_1, BTN_2, BTN_MAIN, BZ?, CN?, D?, J100, J101, J?, K?, LA?, Q?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

Commit message: Kasalar arasi connectorlerin pin cikislari duzenlendi
Parts:
- removed BT?: Battery_Cell, symbol Device:Battery_Cell
- removed BTN_1, BTN_2, BTN_MAIN: SW_Push_Open, symbol Switch:SW_Push_Open
- removed CN?: DIN-2, symbol atlas_robot:DIN-2
- removed D? (x2): LED, symbol Device:LED
- removed J?: DIN-6, symbol Connector:DIN-6
- removed J?: DIN-4, symbol Connector:DIN-4
- removed J?: DIN-7_CenterPin7, symbol Connector:DIN-7_CenterPin7
- removed SW?: OTONOM_MANUAL_SWITCH, symbol atlas_robot:OTONOM_MANUAL_SWITCH
- removed U?: BMS, symbol atlas_robot:BMS
- added BT?: Battery_Cell, symbol Device:Battery_Cell
- added BTN_? (x2), BTN_MAIN? (x2): SW_Push_Open, symbol Switch:SW_Push_Open
- added D?: Otonom Mod LEDi, symbol Device:LED
- added D?: Robot Power Ledi, symbol Device:LED
- added J?: XLR3_Switched, symbol Connector:XLR3_Switched
- added U?: BMS, symbol atlas_robot:BMS
- CN?: value DIN-2 -> ES Kumanda Power
- CN?: value DIN-2 -> PC RESET
- J?: value DIN-4 -> MEGA-IR
- J?: value RJ45 -> BULLET
- J?: value DIN-3 -> GATE
- J? (x2): value DIN-4 -> POWER 24,12,5
- J?: value DIN-3 -> RP POWER
- J?: value DIN-7_CenterPin7 -> SAFETY LIGHTS
- J?: value DB9_Female -> I2C
- J?: value RJ45 -> PC
- J?: value DIN-5 -> HESAI
- J?: value DIN-6 -> CANBUS
- J?: value RJ45 -> HESAI
Connections:
- net CANH_BMS is gone; now on net BMSH: U50.5 (CANH)
- net CANH_CURTIS is gone; now on net CURTISH: U51.5 (CANH)
- net CANL_BMS is gone; now on net BMSL: U50.6 (CANL)
- net CANL_CURTIS is gone; now on net CURTISL: U51.6 (CANL)
- net GREEN ALARM is gone; now on net YESIL: LA?.2 (+), U?. (VCC)
- net PC_ON_HEADER is gone; now on net YESIL: U?. (VCC)
- net PC_ON_HEADER_GND is gone; now on net YESIL: U?. (VCC)
- net +24V: now also BTN_MAIN?.2 (B), U?. (POW_OUT)
- net EMERGENCY: now also BTN_?.2 (B), D?.2 (A), U?. (POW_OUT)
- net GND: now also CN?.2, J?.1, J?.1, J?.1, J?.2, J?.2, J?.3, J?.3, J?.4, BT?.2 (-), D?.1 (K), D?.1 (K)
- net N2HET2_10: now also D?.2 (A), J?.4
- net N2HET2_2/N2HET2_NDIS: now also J?.1
- net N2HET2_9: now also BZ?.1 (-), J?.2
- net SARJ START: no longer D?.2 (A)
- net at CN?.1, U?.3 (COM): now also U?. (POW_OUT)
- net at CN?.2, U?.4 (MANUEL_OTONOM): now also J?.N
- net YESIL: now reaches U?. (VCC)
- net YESIL: now also J?.3
- net MAVİ: now reaches J?.1
- net KAHVE: now reaches J?.2
- net 5V: now reaches J?.2
- net 5V: now also J?.2, J?.3
- net 12V: now reaches J?.3
- net 12V: now also J?.1, J?.3
- net 24V: now reaches J?.4
- net 24V: now also CN?.1, J?.4
- net 9V: now reaches J?.3
- net SARI: now reaches J?.4
- net SARI: now also LA?.2 (+), U?. (VCC)
- net KIRMIZI: now reaches J?.6
- net KIRMIZI: now also LA?.2 (+), U?. (VCC)
- net SDA: now reaches J?.1
- net SCL: now reaches J?.2
- net PC_ON_GND: now reaches CN?.1
- net PC_ON_GND: now also U?. (VCC)
- net PC_ON: now reaches CN?.2
- net PC_ON: now also U?. (VCC)
- net BMSH: now reaches J?.1
- net CURTISH: now reaches J?.2
- net CURTISL: now reaches J?.3
- net BMSL: now reaches J?.5
- removed net BUZZER ALARM: BZ?.1 (-), U?. (VCC)
- removed net RED ALARM: LA?.2 (+), U?. (VCC)
- removed net YELLOW ALARM: LA?.2 (+), U?. (VCC)
- new net: BT?.1 (+), BTN_MAIN?.1 (A), U?. (POW_OUT)
- new net: BTN_?.1 (A), BTN_MAIN?.1 (A)
- new net: D?.2 (A), J?.NO, U?. (POW_OUT)
- new net: BTN_?.1 (A), BTN_?.2 (B)
- new net ALL_ROBOT: BTN_MAIN?.2 (B)
Other:
- note added: "ANA ACİL STOP BURADAKİ İKİ SWITHCI KESER"
- note added: "Emergency Stop Butonları Normade SC Basıldığında OC olarak çalışır"
- note added: "MODE pinleri SC olursa otonom moda geçer OC olursa manuel moddadır Emergency ucu 24V göremezse Bataryayı Kapatır"
- note added: "SW Robot üstünde 3 konum var Sağda-Solda iken: OTONOM (SC) ortada: MANUEL (OC)"
- note added: "Vinç Kumandası Normalde Short Circuit Röle çektiğinde Open Circuit"
- note removed: "MODE pinleri short olursa otonom moda geçer aksi durumda manuel moddadır"
- note removed: "SW Sağda ve Solda iken: OTONOM ortada: MANUEL"
- moved on the sheet: BZ?, CN?, D?, J100, J101, J?, SW?, U50, U51, U?
